File: pcb.kicad_pcb (KiCad board)
At the start: 2 copper layers, 71 x 69.5 mm, 12 parts, among them SW1 SW_Push, U1 NE555P, U2 NE555P

Commit message: PCB_design
Parts:
- D1: footprint LED_SMD:LED_0201_0603Metric -> LED_SMD:LED_0402_1005Metric_Pad0.77x0.64mm_HandSolder
- moved D1 1.00 mm to (175.3, 116.5)
Routing:
- net GND: track 117.6 -> 124.9 mm, vias 0 -> 2
