File: pcb.kicad_sch (KiCad schematic)
At the start: 12 parts, among them SW1 SW_Push, U1 NE555P, U2 NE555P

Commit message: PCB_design
Parts:
- D1: footprint LED_SMD:LED_0201_0603Metric -> LED_SMD:LED_0402_1005Metric_Pad0.77x0.64mm_HandSolder
Changed lines of the file:
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@@
 			)
 		)
-		(property "Footprint" "LED_SMD:LED_0201_0603Metric"
+		(property "Footprint" "LED_SMD:LED_0402_1005Metric_Pad0.77x0.64mm_HandSolder"
 			(at 111.76 93.98 0)
 			(effects
